File: hardware/Mk1/Power_Deck_Longitudinal/Power_Deck_Longitudinal_v0.1.kicad_sch (KiCad schematic)
At the start: 8 parts, among them J1 XT30_IN, J2 INA219_MODULE, J3 MP1584_MODULE, J4 Main Deck Connector, SW1 SW_SPST

Commit message: feat(hardware): add Mk1 longitudinal PCB designs
Parts:
- removed SW1: SW_SPST, symbol Switch:SW_SPST
- added J5: SLED_SWITCH, Connector_JST:JST_XH_B2B-XH-A_1x02_P2.50mm_Vertical, symbol Connector_Generic:Conn_01x02
- C1: value 100 uF 16 V -> 470 uF 16 V; footprint (none) -> Capacitor_THT:CP_Radial_D8.0mm_P3.50mm
- C2: footprint (none) -> Capacitor_THT:C_Disc_D5.0mm_W2.5mm_P5.00mm
- F1: footprint (none) -> RocketOS_Mk1:JK30_200
- J1: footprint (none) -> RocketOS_Mk1:XT30PW_F_RocketOS
- J2: footprint (none) -> RocketOS_Mk1:INA219_MODULE
- J3: footprint (none) -> RocketOS_Mk1:MP1584
- J4: footprint (none) -> Connector_JST:JST_XH_B5B-XH-A_1x05_P2.50mm_Vertical
Connections:
- net GND: now also J1.1 (Pin_1); no longer J1.2 (Pin_2)
- net VBAT: now also J1.2 (Pin_2); no longer J1.1 (Pin_1)
- net VBAT_PROTECTED: now also J5.1 (Pin_1)
- net VBAT_SW: now also J5.2 (Pin_2)
Other:
- note added: "External sled power switch"
- moved on the sheet: J1
