File: hardware/Mk1/Main_Deck_Longitudinal_v0.1/Main_Deck_Longitudinal_v0.1.kicad_pcb (KiCad board)
At the start: 2 copper layers, 30 x 85.5 mm, 11 parts, among them J1 BMP388, J2 NEO-M9N, J3 Micro SD, J4 Power Deck, J5 GY-87, J7 Active Buzzer(5V), Q1 S8050, U1 Ai-Thinker-Ra-02, U2 ESP32-S3_MINI_Nano_N16R8

Commit message: fix(hardware): resolve Mk1 I2C address collision
Connections:
- J1 pad 5: unconnected-(J1-Pin_5-Pad5) -> GND
Routing:
- net GND: track 4.25 -> 10.9 mm
