File: hardware/Mk1/Main_Deck_Longitudinal_v0.1/Main_Deck_Longitudinal_v0.1.kicad_sch (KiCad schematic)
At the start: 11 parts, among them J1 BMP388, J2 NEO-M9N, J3 Micro SD, J4 Power Deck, J5 GY-87, J7 Active Buzzer(5V), Q1 S8050, U1 Ai-Thinker-Ra-02, U2 ESP32-S3_MINI_Nano_N16R8

Commit message: fix(hardware): resolve Mk1 I2C address collision
Connections:
- net GND: now also J1.5 (Pin_5)
- no-connect marks 39 -> 38
Changed lines of the file:
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@@
-	)
-	(no_connect
-		(at 259.08 27.94)
 	)
 	(no_connect
@@
 		(pts
 			(xy 138.43 68.58) (xy 144.78 68.58)
+		)
+		(stroke
+			(width 0)
+			(type default)
+		)
+	)
+	(wire
+		(pts
+			(xy 248.92 27.94) (xy 259.08 27.94)
 		)
 		(stroke
@@
 					(unit 1)
 				)
+			)
+		)
+	)
+	(symbol
+		(lib_id "power:GND")
+		(at 248.92 27.94 270)
+		(unit 1)
+		(body_style 1)
+		(exclude_from_sim no)
+		(in_bom yes)
+		(on_board yes)
+		(in_pos_files yes)
+		(dnp no)
+		(fields_autoplaced yes)
+		(property "Reference" "#PWR017"
+			(at 242.57 27.94 0)
+			(hide yes)
+			(show_name no)
+			(do_not_autoplace no)
+			(effects
+				(font
+					(size 1.27 1.27)
+				)
+			)
+		)
+		(property "Value" "GND"
+			(at 245.11 27.9399 90)
+			(show_name no)
+			(do_not_autoplace no)
+			(effects
+				(font
+					(size 1.27 1.27)
+				)
+				(justify right)
+			)
+		)
+		(property "Footprint" ""
+			(at 248.92 27.94 0)
+			(hide yes)
+			(show_name no)
+			(do_not_autoplace no)
+			(effects
+				(font
+					(size 1.27 1.27)
+				)
+			)
+		)
+		(property "Datasheet" ""
+			(at 248.92 27.94 0)
+			(hide yes)
+			(show_name no)
+			(do_not_autoplace no)
+			(effects
+				(font
+					(size 1.27 1.27)
+				)
+			)
+		)
+		(property "Description" "Power symbol creates a global label with name \"GND\" , ground"
+			(at 248.92 27.94 0)
+			(hide yes)
+			(show_name no)
+			(do_not_autoplace no)
+			(effects
+				(font
+					(size 1.27 1.27)
+				)
+			)
+		)
+		(pin "1"
+		)
+		(instances
+			(project "Main_Deck_Longitudinal_v0.1"
+				(path "/e31ac7f1-555d-4190-a97f-833d688a3009"
+					(reference "#PWR017")
+					(unit 1)
+				)
